Commit message: urdf directory change

File: Project_1/src/pr_config/urdf_files/pr.urdf (robot description, URDF)
Before this commit: robot origins, 3 links, 2 joints
Joints:
- joint p: limit lower=-1 upper=0 effort=1000.0 velocity=0.5 -> lower=-1 upper=0 effort=1000.0 velocity=1.5
- joint r: limit lower=-3.14 upper=3.14 effort=1000.0 velocity=0.5 -> lower=-3.14 upper=3.14 effort=1000.0 velocity=1.5
